File: KiCad/GitKop/GitKop.kicad_sch (KiCad schematic)
At the start: 18 parts, among them J1 Conn_01x02_Socket, J2 Conn_01x02_Socket, J3 Conn_01x02_Socket, Q1 BC557, Q2 BC547, Q3 IRF740, U1 TL071, U2 TL071, U3 LF356

Commit message: x
Parts:
- added R7: 2000, symbol Device:R
Connections:
- net at C1.2: now also R7.1
Other:
- moved on the sheet: U2
Changed lines of the file:
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@@
 (kicad_sch
-	(version 20231120)
+	(version 20250114)
 	(generator "eeschema")
-	(generator_version "8.0")
+	(generator_version "9.0")
 	(paper "A4")
 	(title_block
@@
 	(wire
 		(pts
-			(xy 177.8 77.47) (xy 177.8 81.28)
-		)
-		(stroke
-			(width 0)
-			(type default)
-		)
-	)
-	(wire
-		(pts
-			(xy 177.8 58.42) (xy 177.8 62.23)
+			(xy 177.8 66.04) (xy 177.8 69.85)
+		)
+		(stroke
+			(width 0)
+			(type default)
+		)
+	)
+	(wire
+		(pts
+			(xy 177.8 46.99) (xy 177.8 50.8)
 		)
 		(stroke
@@
 		(pts
 			(xy 176.53 93.98) (xy 176.53 97.79)
+		)
+		(stroke
+			(width 0)
+			(type default)
+		)
+	)
+	(wire
+		(pts
+			(xy 166.37 102.87) (xy 166.37 113.03)
 		)
 		(stroke
@@
 	(global_label "VCC"
 		(shape input)
-		(at 177.8 58.42 0)
+		(at 177.8 46.99 0)
 		(fields_autoplaced yes)
 		(effects
@@
 		)
 		(property "Intersheetrefs" "${INTERSHEET_REFS}"
-			(at 184.4138 58.42 0)
+			(at 184.4138 46.99 0)
 			(effects
 				(font
@@
 		(on_board yes)
 		(dnp no)
-		(fields_autoplaced yes)
 		(property "Reference" "D2"
 			(at 152.4 115.5699 90)
@@
 		)
 		(property "Value" "BAV19"
-			(at 152.4 118.1099 90)
+			(at 152.4 118.1099 0)
 			(effects
 				(font
@@
 	)
 	(symbol
+		(lib_id "Device:R")
+		(at 166.37 116.84 0)
+		(unit 1)
+		(exclude_from_sim no)
+		(in_bom yes)
+		(on_board yes)
+		(dnp no)
+		(fields_autoplaced yes)
+		(property "Reference" "R7"
+			(at 168.91 115.5699 0)
+			(effects
+				(font
+					(size 1.27 1.27)
+				)
+				(justify left)
+			)
+		)
+		(property "Value" "2000"
+			(at 168.91 118.1099 0)
+			(effects
+				(font
+					(size 1.27 1.27)
+				)
+				(justify left)
+			)
+		)
+		(property "Footprint" ""
+			(at 164.592 116.84 90)
+			(effects
+				(font
+					(size 1.27 1.27)
+				)
+				(hide yes)
+			)
+		)
+		(property "Datasheet" "~"
+			(at 166.37 116.84 0)
+			(effects
+				(font
+					(size 1.27 1.27)
+				)
+				(hide yes)
+			)
+		)
+		(property "Description" "Resistor"
+			(at 166.37 116.84 0)
+			(effects
+				(font
+					(size 1.27 1.27)
+				)
+				(hide yes)
+			)
+		)
+		(pin "2"
+		)
+		(pin "1"
+		)
+		(instances
+			(project "GitKop"
+				(path "/cf516f6b-7df6-4407-90f1-f14d517be13f"
+					(reference "R7")
+					(unit 1)
+				)
+			)
+		)
+	)
+	(symbol
 		(lib_id "Amplifier_Operational:LF356")
 		(at 179.07 105.41 0)
@@
 	(symbol
 		(lib_id "power:GND")
-		(at 177.8 81.28 0)
+		(at 177.8 69.85 0)
 		(unit 1)
 		(exclude_from_sim no)
@@
 		(fields_autoplaced yes)
 		(property "Reference" "#PWR02"
-			(at 177.8 87.63 0)
+			(at 177.8 76.2 0)
 			(effects
 				(font
@@
 		)
 		(property "Value" "GND"
-			(at 177.8 86.36 0)
+			(at 177.8 74.93 0)
 			(effects
 				(font
@@
 		)
 		(property "Footprint" ""
-			(at 177.8 81.28 0)
+			(at 177.8 69.85 0)
 			(effects
 				(font
@@
 		)
 		(property "Datasheet" ""
-			(at 177.8 81.28 0)
+			(at 177.8 69.85 0)
 			(effects
 				(font
@@
 		)
 		(property "Description" "Power symbol creates a global label with name \"GND\" , ground"
-			(at 177.8 81.28 0)
+			(at 177.8 69.85 0)
 			(effects
 				(font
@@
 	(symbol
 		(lib_id "Amplifier_Operational:TL071")
-		(at 180.34 69.85 0)
+		(at 180.34 58.42 0)
 		(unit 1)
 		(exclude_from_sim no)
@@
 		(fields_autoplaced yes)
 		(property "Reference" "U2"
-			(at 189.23 63.5314 0)
+			(at 189.23 52.1014 0)
 			(effects
 				(font
@@
 		)
 		(property "Value" "TL071"
-			(at 189.23 66.0714 0)
+			(at 189.23 54.6414 0)
 			(effects
 				(font
@@
 		)
 		(property "Footprint" ""
-			(at 181.61 68.58 0)
+			(at 181.61 57.15 0)
 			(effects
 				(font
@@
 		)
 		(property "Datasheet" "http://www.ti.com/lit/ds/symlink/tl071.pdf"
-			(at 184.15 66.04 0)
+			(at 184.15 54.61 0)
 			(effects
 				(font
@@
 		)
 		(property "Description" "Single Low-Noise JFET-Input Operational Amplifiers, DIP-8/SOIC-8"
-			(at 180.34 69.85 0)
+			(at 180.34 58.42 0)
 			(effects
 				(font
@@
 		)
 	)
+	(embedded_fonts no)
 )

Commit message: Update GitKop.kicad_sch
Parts:
- added D3: 3.3V, symbol Device:D_Zener
Connections:
- net GND: now also D3.2 (A)
- net SIGNAL_OUT: now also U1.6, D3.1 (K)
Other:
- moved on the sheet: U2, U3

Commit message: pierwszy schemat
Parts:
- added R10: 2000, symbol Device:R
- added R11, R8, R9: 1000, symbol Device:R
- added R12: 1M, symbol Device:R
- added R13: 1k, symbol Device:R
Connections:
- net COIL2: now also R9.1
- net GND: now also R10.2, R13.2, R8.2
- net SIGNAL_OUT: now also U1.2 (-)
- net at C1.2, R7.1: now also U2.3 (+)
- net VGND: now reaches R7.2
- net VGND: now also U3.2 (-), U3.6
- net at U3.3 (+): now also R8.1, R9.2
- net at U1.3 (+): now also R10.1, R11.2
- net at U2.2 (-): now also R12.1, R13.1
- net at U2.6: now also R11.1, R12.2
Other:
- moved on the sheet: D3, J1, J2, J3, U1, U2, U3

Commit message: kicad: update
Parts:
- R10: value 2000 -> 1000
- R11: value 1000 -> 2000
- U1: value TL071 -> MCP6281
- U3: value LF356 -> TL071
Changed lines of the file:
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@@
 			)
 		)
-		(property "Value" "2000"
+		(property "Value" "1000"
 			(at 219.71 113.0299 0)
 			(effects
@@
 		(fields_autoplaced yes)
 		(property "Reference" "U3"
-			(at 130.81 57.1814 0)
-			(effects
-				(font
-					(size 1.27 1.27)
-				)
-			)
-		)
-		(property "Value" "LF356"
-			(at 130.81 59.7214 0)
+			(at 130.81 57.0798 0)
+			(effects
+				(font
+					(size 1.27 1.27)
+				)
+			)
+		)
+		(property "Value" "TL071"
+			(at 130.81 59.6198 0)
 			(effects
 				(font
@@
 			)
 		)
-		(property "Value" "1000"
+		(property "Value" "2000"
 			(at 219.71 100.3299 0)
 			(effects
@@
 		(fields_autoplaced yes)
 		(property "Reference" "U1"
-			(at 246.38 101.6314 0)
-			(effects
-				(font
-					(size 1.27 1.27)
-				)
-			)
-		)
-		(property "Value" "TL071"
-			(at 246.38 104.1714 0)
-			(effects
-				(font
+			(at 248.92 101.5298 0)
+			(effects
+				(font
+					(size 1.27 1.27)
+				)
+			)
+		)
+		(property "Value" "MCP6281"
+			(at 248.92 104.0698 0)
+			(effects
+				(font

Commit message: KiCad: Update before ordering
Parts:
- removed J2, J3: Conn_01x02_Socket, symbol Connector:Conn_01x02_Socket
- removed R6: 510, symbol Device:R
- added 1: U1, STM32F4x1CxU6 CoreBoard WeActStudio:STM32F4x1CxU6 WeActStudio, symbol STM32F4x1CxU6 CoreBoard WeActStudio:STM32F4x1CxU6 WeActStudio
- added BZ1: Buzzer, Buzzer_Beeper:Buzzer_12x9.5RM7.6, symbol Device:Buzzer
- added C2, C5: 100uF, Capacitor_THT:CP_Radial_D6.3mm_P2.50mm, symbol Device:C_Polarized
- added C3, C4: 1500uF, Capacitor_THT:CP_Radial_D10.0mm_P5.00mm, symbol Device:C_Polarized
- added J2: Conn_01x08_Socket, Connector_PinSocket_2.54mm:PinSocket_1x08_P2.54mm_Vertical, symbol Connector:Conn_01x08_Socket
- added J3: Conn_01x04_Socket, Connector_PinSocket_2.54mm:PinSocket_1x04_P2.54mm_Vertical, symbol Connector:Conn_01x04_Socket
- added J4: RJ45, MTJ-881X1:MTJ881X1, symbol Connector:RJ45
- added RV1: R_Potentiometer_Trim, Potentiometer_THT:Potentiometer_Bourns_3296W_Vertical, symbol Device:R_Potentiometer_Trim
- added SW1: RotaryEncoder_Switch, Rotary_Encoder:RotaryEncoder_Bourns_Vertical_PEC12R-3x17F-Sxxxx, symbol Device:RotaryEncoder_Switch
- added U4: LF33_TO252, Package_TO_SOT_SMD:TO-252-2, symbol Regulator_Linear:LF33_TO252
- C1: footprint (none) -> Capacitor_SMD:C_1206_3216Metric_Pad1.33x1.80mm_HandSolder
- D3: footprint (none) -> Diode_SMD:D_MiniMELF_Handsoldering
- J1: value Conn_01x02_Socket -> POWER_Socket; footprint (none) -> Connector_BarrelJack:BarrelJack_Horizontal
- R1, R10, R11, R12, R13, R2, R3, R4, R5, R7, R8, R9: footprint (none) -> Resistor_SMD:R_1206_3216Metric_Pad1.30x1.75mm_HandSolder
- U1, U2: footprint (none) -> Package_DIP:DIP-8_W7.62mm_Socket_LongPads
- U3: footprint (none) -> Package_SO:SOIC-8_5.3x5.3mm_P1.27mm
Connections:
- net COIL1: now also J4.5, J4.6, J4.7, J4.8, RV1.3
- net COIL2: now also C3.1, C4.1, C5.1, J4.1, J4.2, J4.3, J4.4, U4.1 (VI)
- net GND: now also 1.39 (GND), BZ1.2 (-), C2.2, C3.2, C4.2, C5.2, J2.2 (Pin_2), J3.1 (Pin_1), SW1.S2, U4.2 (GND)
- net PULSE_IN: now also 1.7 (PA10)
- net SIGNAL_OUT: now also 1.26 (PA0)
- net at C1.1, D1.1 (K), D2.2 (A): now also RV1.2
- new net 3_3V: 1.20 (3V3), C2.1, J2.1 (Pin_1), J2.8 (Pin_8), J3.2 (Pin_2), SW1.C, U4.3 (VO)
- new net BUZZER: 1.10 (PA15), BZ1.1 (+)
- new net ENC_A: 1.35 (PB1), SW1.A
- new net ENC_B: 1.6 (PA9), SW1.B
- new net ENC_BTN: 1.5 (PA8), SW1.S1
- new net I2C_SCL: 1.14 (PB6), J3.3 (Pin_3)
- new net I2C_SDA: 1.37 (PB10), J3.4 (Pin_4)
- new net LCD_CS: J2.3 (Pin_3)
- new net LCD_DC: 1.31 (PA5), J2.5 (Pin_5)
- new net LCD_MOSI: 1.30 (PA4), J2.6 (Pin_6)
- new net LCD_RST: 1.29 (PA3), J2.4 (Pin_4)
- new net LCD_SCK: 1.28 (PA2), J2.7 (Pin_7)
Other:
- title: GitKop - PI Module -> GitKop
- moved on the sheet: C1, D1, D2, D3, J1, Q1, Q2, Q3, R1, R10, R11, R12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

Commit message: gitkop001
Parts:
- added C6, C7, C8: 100uF, Capacitor_THT:CP_Radial_D6.3mm_P2.50mm, symbol Device:C_Polarized
Connections:
- net BUZZER: now also 1.4 (PB15); no longer 1.10 (PA15)
- net COIL2: now also C6.1, C7.1, C8.1
- net GND: now also 1.19 (GND), C6.2, C7.2, C8.2
- net LCD_CS: now also 1.31 (PA5)
- net LCD_DC: now also 1.32 (PA6); no longer 1.31 (PA5)

Commit message: kicad: 1st version
Parts:
- added R6: 1000, Resistor_SMD:R_1206_3216Metric_Pad1.30x1.75mm_HandSolder, symbol Device:R
Connections:
- net COIL1: now also R6.1
- net COIL2: now also RV1.1
- net GND: no longer R13.2
- net VGND: now also R13.2
- net at C1.1, D1.1 (K), D2.2 (A): now also R6.2; no longer RV1.2
Other:
- moved on the sheet: J1, R13, RV1

Commit message: sch: Sprzatanie
Parts:
- RV1: value R_Potentiometer_Trim -> R_Trim
Connections:
- net at C1.2, R7.1, U2.3 (+): now also U2.8 (NC)
Other:
- moved on the sheet: BZ1, D1, D2, R6, R7, RV1
