File: KiCad/GitKop/GitKop.kicad_pcb (KiCad board)
At the start: 2 copper layers, 5 parts, among them Q1 BC557, Q2 BC547, Q3 IRF740

Commit message: KiCad: Update before ordering
Parts:
- added 1: U1, STM32F4x1CxU6 CoreBoard WeActStudio:STM32F4x1CxU6 WeActStudio, F.Cu at (127.5, 45.5)
- added BZ1: Buzzer, Buzzer_Beeper:Buzzer_12x9.5RM7.6, F.Cu at (132.2, 65.0)
- added C1: 1u, Capacitor_SMD:C_1206_3216Metric_Pad1.33x1.80mm_HandSolder, F.Cu at (173.2, 107.8)
- added C2: 100uF, Capacitor_THT:CP_Radial_D6.3mm_P2.50mm, F.Cu at (137.5, 31.5)
- added C3: 1500uF, Capacitor_THT:CP_Radial_D10.0mm_P5.00mm, F.Cu at (148.4, 91.4)
- added C4: 1500uF, Capacitor_THT:CP_Radial_D10.0mm_P5.00mm, F.Cu at (199.0, 112.5)
- added C5: 100uF, Capacitor_THT:CP_Radial_D6.3mm_P2.50mm, F.Cu at (104.2, 63.0)
- added D3: 3.3V, Diode_SMD:D_MiniMELF_Handsoldering, F.Cu at (143.0, 146.2)
- added J1: POWER_Socket, Connector_BarrelJack:BarrelJack_Horizontal, F.Cu at (193.0, 94.5)
- added J2: Conn_01x08_Socket, Connector_PinSocket_2.54mm:PinSocket_1x08_P2.54mm_Vertical, F.Cu at (130.5, 32.0)
- added J3: Conn_01x04_Socket, Connector_PinSocket_2.54mm:PinSocket_1x04_P2.54mm_Vertical, F.Cu at (176.0, 87.9)
- added J4: RJ45, MTJ-881X1:MTJ881X1, F.Cu at (183.7, 74.7)
- added R1: 100, Resistor_SMD:R_1206_3216Metric_Pad1.30x1.75mm_HandSolder, F.Cu at (92.5, 93.5)
- added R10: 1000, Resistor_SMD:R_1206_3216Metric_Pad1.30x1.75mm_HandSolder, F.Cu at (117.0, 150.6)
- added R11: 2000, Resistor_SMD:R_1206_3216Metric_Pad1.30x1.75mm_HandSolder, F.Cu at (117.0, 143.9)
- added R12: 1M, Resistor_SMD:R_1206_3216Metric_Pad1.30x1.75mm_HandSolder, F.Cu at (144.4, 136.0)
- added R13: 1k, Resistor_SMD:R_1206_3216Metric_Pad1.30x1.75mm_HandSolder, F.Cu at (131.4, 134.5)
- added R2: 1000, Resistor_SMD:R_1206_3216Metric_Pad1.30x1.75mm_HandSolder, F.Cu at (68.0, 85.5)
- added R3: 1000, Resistor_SMD:R_1206_3216Metric_Pad1.30x1.75mm_HandSolder, F.Cu at (108.0, 119.1)
- added R4: 6800, Resistor_SMD:R_1206_3216Metric_Pad1.30x1.75mm_HandSolder, F.Cu at (76.5, 77.5)
- added R5: 2000, Resistor_SMD:R_1206_3216Metric_Pad1.30x1.75mm_HandSolder, F.Cu at (114.0, 112.5)
- added R7: 2000, Resistor_SMD:R_1206_3216Metric_Pad1.30x1.75mm_HandSolder, F.Cu at (114.0, 115.8)
- added R8: 1000, Resistor_SMD:R_1206_3216Metric_Pad1.30x1.75mm_HandSolder, F.Cu at (166.5, 140.0)
- added R9: 1000, Resistor_SMD:R_1206_3216Metric_Pad1.30x1.75mm_HandSolder, F.Cu at (174.0, 135.0)
- added RV1: R_Potentiometer_Trim, Potentiometer_THT:Potentiometer_Bourns_3296W_Vertical, F.Cu at (133.0, 97.5)
- added SW1: RotaryEncoder_Switch, Rotary_Encoder:RotaryEncoder_Bourns_Vertical_PEC12R-3x17F-Sxxxx, F.Cu at (72.0, 119.0)
- added U1: MCP6281, Package_DIP:DIP-8_W7.62mm_Socket_LongPads, F.Cu at (136.5, 151.0)
- added U2: TL071, Package_DIP:DIP-8_W7.62mm_Socket_LongPads, F.Cu at (136.7, 121.4)
- added U3: TL071, Package_SO:SOIC-8_5.3x5.3mm_P1.27mm, F.Cu at (166.0, 134.5)
- added U4: LF33_TO252, Package_TO_SOT_SMD:TO-252-2, F.Cu at (99.5, 30.7)
- moved D1 72.8 mm to (115.8, 94.5), turned to 180 degrees
- moved Q3 54.1 mm to (105.1, 82.0), turned to 180 degrees
- moved D2 51.2 mm to (108.2, 88.5), turned to 0 degrees
- moved Q1 27.2 mm to (90.5, 85.5)
- moved Q2 22.0 mm to (77.0, 86.0)

Commit message: kicad: 0th version
Parts:
- moved R2 115.2 mm to (161.0, 153.4), turned to -90 degrees
- moved R4 110.7 mm to (157.0, 153.4), turned to 90 degrees
- moved Q2 110.3 mm to (157.5, 161.4)
- moved J4 98.1 mm to (130.3, 157.1), turned to -90 degrees
- moved R1 97.4 mm to (156.9, 166.5), turned to 180 degrees
- moved Q1 96.7 mm to (150.2, 161.5)
- moved U4 85.8 mm to (163.5, 87.8), turned to 0 degrees
- moved C4 77.7 mm to (121.5, 117.9), turned to 90 degrees
- moved J1 75.2 mm to (127.0, 130.5), turned to 0 degrees
- moved SW1 74.9 mm to (144.7, 101.3), turned to -90 degrees
- moved Q3 72.5 mm to (140.0, 145.5)
- moved C2 70.8 mm to (121.5, 100.5), turned to -90 degrees
- moved R5 64.6 mm to (149.4, 166.5)
- moved RV1 63.4 mm to (140.5, 160.5), turned to 90 degrees
- moved C3 61.2 mm to (122.5, 146.9), turned to 90 degrees
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Other:
- board outline added: 58.5 x 126.5 mm

Commit message: gitkop001
Parts:
- added C6: 100uF, Capacitor_THT:CP_Radial_D6.3mm_P2.50mm, F.Cu at (184.5, 125.0)
- added C7: 100uF, Capacitor_THT:CP_Radial_D6.3mm_P2.50mm, F.Cu at (174.5, 156.5)
- added C8: 100uF, Capacitor_THT:CP_Radial_D6.3mm_P2.50mm, F.Cu at (138.0, 132.0)
- moved C5 66.9 mm to (184.5, 114.5)
- moved C2 63.1 mm to (184.5, 104.5), turned to 0 degrees
- moved BZ1 47.3 mm to (121.5, 98.9), turned to -90 degrees
- moved R1 46.7 mm to (132.0, 127.0), turned to 90 degrees
- moved J3 46.0 mm to (158.2, 103.0)
- moved Q2 44.4 mm to (139.0, 121.0)
- moved Q1 44.4 mm to (131.8, 121.1)
- moved R2 44.4 mm to (142.5, 113.1)
- moved R3 44.4 mm to (133.0, 114.6)
- moved R4 42.9 mm to (138.0, 115.0), turned to -90 degrees
- moved R13 35.8 mm to (183.0, 145.1)
- moved R12 35.4 mm to (183.0, 151.1), turned to -90 degrees
- moved U2 26.4 mm to (177.0, 144.4)
- moved D3 25.8 mm to (160.5, 128.0), turned to 180 degrees
- moved U1 24.9 mm to (169.2, 128.8)
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Connections:
- 1 pad 10: BUZZER -> unconnected-(1A-PA15-Pad10)
- 1 pad 19: unconnected-(1A-GND-Pad19) -> GND
- 1 pad 31: LCD_DC -> LCD_CS
- 1 pad 32: unconnected-(1A-PA6-Pad32) -> LCD_DC
- 1 pad 4: unconnected-(1A-PB15-Pad4) -> BUZZER
Routing:
- net COIL2: track 0.00 -> 264.9 mm
- net 3_3V: track 0.00 -> 164.7 mm
- net ENC_A: track 0.00 -> 94.1 mm, vias 0 -> 8
- net SIGNAL_OUT: track 0.00 -> 68.5 mm, vias 0 -> 4
- net LCD_SCK: track 0.00 -> 45.8 mm
- net ENC_BTN: track 0.00 -> 42.0 mm
- net COIL1: track 0.00 -> 40.7 mm
- net LCD_RST: track 0.00 -> 40.2 mm, vias 0 -> 2
- net LCD_MOSI: track 0.00 -> 39.7 mm
- net Net-(R11-Pad1): track 0.00 -> 38.0 mm
- net I2C_SDA: track 0.00 -> 37.2 mm, vias 0 -> 2
- net LCD_CS: track 0.00 -> 34.1 mm, vias 0 -> 2
- net LCD_DC: track 0.00 -> 33.6 mm
- net ENC_B: track 0.00 -> 25.1 mm
- net PULSE_IN: track 0.00 -> 24.5 mm, vias 0 -> 2
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- added copper zone on B.Cu, net GND
- added copper zone on F.Cu, net GND
Other:
- board size 58.5 x 126.5 mm -> 80 x 101 mm
- board text added: "GitKop 001"
- board text added: "gitmanik.dev Pawel Reich 2025"

Commit message: kicad: updated
Parts:
- added R6: 1000, Resistor_SMD:R_1206_3216Metric_Pad1.30x1.75mm_HandSolder, F.Cu at (159.3, 154.0)
- RV1: value R_Potentiometer_Trim -> R_Trim
- moved RV1 19.2 mm to (142.0, 146.0)
- moved C1 5.83 mm to (159.3, 147.5)
- moved D1 5.83 mm to (155.1, 147.5)
- moved D2 5.83 mm to (147.5, 141.5)
- moved R7 5.83 mm to (159.3, 141.0)
- moved Q3 5.04 mm to (153.5, 156.1)
Connections:
- R13 pad 2: GND -> VGND
- RV1 pad 1: unconnected-(RV1-Pad1) -> COIL2
- RV1 pad 2: Net-(D1-K) -> COIL1
- RV1 pad 3: COIL1 -> unconnected-(RV1-Pad3)
Routing:
- net Net-(Q1-C): track 4.41 -> 47.1 mm, vias 0 -> 1
- net VGND: track 15.9 -> 43.7 mm
- net COIL2: track 264.9 -> 273.3 mm
- net Net-(U2-+): track 23.8 -> 17.7 mm
- net Net-(D1-K): track 20.7 -> 14.7 mm
- net COIL1: track 40.7 -> 44.9 mm

Commit message: sch: fix mcp6281 vcc
Parts:
- R5: value 2000 -> 170
- R6: value 1000 -> 3100
Connections:
- C6 pad 1: COIL2 -> 3_3V
- U1 pad 7: COIL2 -> 3_3V
Routing:
- net 3_3V: track 164.7 -> 185.0 mm, vias 0 -> 2
- net COIL2: track 273.3 -> 262.6 mm
Changed lines of the file:
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@@
 			(psnegative no)
 			(psa4output no)
-			(plot_black_and_white yes)
+			(plot_black_and_white no)
 			(sketchpadsonfab no)
 			(plotpadnumbers no)
@@
 			(crossoutdnponfab yes)
 			(subtractmaskfromsilk no)
-			(outputformat 1)
+			(outputformat 5)
 			(mirror no)
 			(drillshape 0)
 			(scaleselection 1)
-			(outputdirectory "gerber/")
+			(outputdirectory "../../doc/img/pcb/")
 		)
 	)
@@
 			)
 		)
-		(property "Value" "1000"
+		(property "Value" "3100"
 			(at 0 1.83 90)
 			(layer "F.Fab")
@@
 			)
 		)
-		(property "Value" "2000"
+		(property "Value" "170"
 			(at 0 1.83 90)
 			(layer "F.Fab")
@@
 			(layers "*.Cu" "*.Mask")
 			(remove_unused_layers no)
-			(net 2 "COIL2")
+			(net 16 "3_3V")
 			(pinfunction "V+")
 			(pintype "power_in")
@@
 			(remove_unused_layers no)
 			(roundrect_rratio 0.15625)
-			(net 2 "COIL2")
+			(net 16 "3_3V")
 			(pintype "passive")
 		)
@@
 	)
 	(segment
-		(start 171.73 118.15)
-		(end 177.125 112.755)
-		(width 0.5)
-		(layer "F.Cu")
-		(net 2)
-	)
-	(segment
 		(start 137.14 146.31)
 		(end 137.5 145.95)
@@
 	)
 	(segment
-		(start 171.73 121.19)
-		(end 171.73 118.15)
-		(width 0.5)
-		(layer "F.Cu")
-		(net 2)
-	)
-	(segment
 		(start 130 145.04)
 		(end 128.46 145.04)
@@
 	)
 	(segment
+		(start 180 110)
+		(end 180 108.195)
+		(width 0.5)
+		(layer "F.Cu")
+		(net 16)
+	)
+	(segment
 		(start 182 87)
 		(end 182 73)
@@
 	)
 	(segment
+		(start 171.73 116.77)
+		(end 172.5 116)
+		(width 0.5)
+		(layer "F.Cu")
+		(net 16)
+	)
+	(segment
+		(start 172.5 116)
+		(end 179 116)
+		(width 0.5)
+		(layer "F.Cu")
+		(net 16)
+	)
+	(segment
 		(start 184.5 96.1308)
 		(end 184.5 104.5)
@@
 	)
 	(segment
+		(start 179 116)
+		(end 180 115)
+		(width 0.5)
+		(layer "F.Cu")
+		(net 16)
+	)
+	(segment
 		(start 179.5846 89.4154)
 		(end 182 87)
@@
 	)
 	(segment
-		(start 177.125 108.195)
+		(start 180 108.195)
 		(end 180.805 108.195)
 		(width 0.5)
@@
 	)
 	(segment
+		(start 177.125 108.195)
+		(end 180 108.195)
+		(width 0.5)
+		(layer "F.Cu")
+		(net 16)
+	)
+	(segment
+		(start 180 115)
+		(end 179.951 114.951)
+		(width 0.5)
+		(layer "F.Cu")
+		(net 16)
+	)
+	(segment
+		(start 171.73 118.15)
+		(end 171.73 116.77)
+		(width 0.5)
+		(layer "F.Cu")
+		(net 16)
+	)
+	(segment
 		(start 177.7846 89.4154)
 		(end 179.5846 89.4154)
@@
 	)
 	(segment
+		(start 171.73 121.19)
+		(end 171.73 118.15)
+		(width 0.5)
+		(layer "F.Cu")
+		(net 16)
+	)
+	(segment
 		(start 154 108.6)
 		(end 154 105.5)
@@
 		(net 16)
 	)
+	(via
+		(at 180 115)
+		(size 0.6)
+		(drill 0.3)
+		(layers "F.Cu" "B.Cu")
+		(net 16)
+	)
+	(via
+		(at 180 110)
+		(size 0.6)
+		(drill 0.3)
+		(layers "F.Cu" "B.Cu")
+		(net 16)
+	)
 	(segment
 		(start 120.5 74.26)
@@
 	)
 	(segment
+		(start 180 115)
+		(end 180 110)
+		(width 0.5)
+		(layer "B.Cu")
+		(net 16)
+	)
+	(segment
 		(start 121.76 74.26)
 		(end 123.5 76)
@@
 		(polygon
 			(pts
-				(xy 112.5 64) (xy 198.5 64) (xy 197 174) (xy 105.5 173) (xy 107 64.5)
+				(xy 112 65.5) (xy 197.5 66) (xy 198 172.5) (xy 109 171.5) (xy 111.5 65.5)
 			)
 		)
